File: hardware/wearable_revA/wearable_revA.kicad_sch (KiCad schematic)
At the start: 0 parts

Commit message: Update Rev A schematic Include screenshot for proof
Parts:
- added J1, J2: Conn_01x15_Socket, symbol Connector:Conn_01x15_Socket
- added J3: Conn_01x02_Pin, symbol Connector:Conn_01x02_Pin
- added R1, R2: 4.7k, symbol Device:R_US
Connections:
- new net +3.3V: J2.15 (Pin_15), J3.1 (Pin_1), R1.2, R2.2
- new net GND: J2.14 (Pin_14), J3.2 (Pin_2)
- new net SCL: J2.2 (Pin_2), R2.1
- new net SDA: J2.5 (Pin_5), R1.1
Other:
- company: (none) -> University of Rochester
- title: (none) -> Wearable Health Monitor

Commit message: Update schematic design Update log.md
Parts:
- added C1: 10µF, symbol Device:C
- added C2: 0.1µF, symbol Device:C
- added J4: OLED_I2C, symbol Connector:Conn_01x04_Pin
- added J5: MAX30102, symbol Connector:Conn_01x06_Pin
- added TP1: TP_3V3, symbol Connector:TestPoint
- added TP2: TP_GND, symbol Connector:TestPoint
- added TP3: TP_SDA, symbol Connector:TestPoint
- added TP4: TP_SCL, symbol Connector:TestPoint
- J1: value Conn_01x15_Socket -> ESP32 Col1
- J2: value Conn_01x15_Socket -> ESP32 Col2
Connections:
- net +3.3V: now also C1.1, C2.1, J4.2 (Pin_2), J5.1 (Pin_1), TP1.1
- net GND: now also C1.2, C2.2, J4.1 (Pin_1), J5.2 (Pin_2), TP2.1
- net SCL: now also J4.3 (Pin_3), J5.3 (Pin_3), TP4.1
- net SDA: now also J4.4 (Pin_4), J5.4 (Pin_4), TP3.1
- no-connect marks 0 -> 28
Other:
- moved on the sheet: J2, J3, R1, R2

Commit message: Finalize Rev A PCB design Update log.md
Parts:
- C1, C2: footprint (none) -> Capacitor_SMD:C_0603_1608Metric
- J1, J2: footprint (none) -> Connector_PinSocket_2.54mm:PinSocket_1x15_P2.54mm_Vertical
- J3: footprint (none) -> Connector_PinHeader_2.54mm:PinHeader_1x02_P2.54mm_Vertical
- J4: footprint (none) -> Connector_PinHeader_2.54mm:PinHeader_1x04_P2.54mm_Vertical
- J5: footprint (none) -> Connector_PinHeader_2.54mm:PinHeader_1x06_P2.54mm_Vertical
- R1, R2: footprint (none) -> Resistor_SMD:R_0603_1608Metric
- TP1, TP2: footprint (none) -> TestPoint:TestPoint_Loop_D2.50mm_Drill1.0mm
- TP3, TP4: footprint (none) -> TestPoint:TestPoint_Pad_D1.5mm
Changed lines of the file:
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@@
 			)
 		)
-		(property "Footprint" ""
+		(property "Footprint" "Resistor_SMD:R_0603_1608Metric"
 			(at 209.804 98.044 90)
 			(effects
@@
 			)
 		)
-		(property "Footprint" ""
+		(property "Footprint" "Connector_PinSocket_2.54mm:PinSocket_1x15_P2.54mm_Vertical"
 			(at 179.07 114.3 0)
 			(effects
@@
 			)
 		)
-		(property "Footprint" ""
+		(property "Footprint" "Connector_PinHeader_2.54mm:PinHeader_1x02_P2.54mm_Vertical"
 			(at 161.29 148.59 0)
 			(effects
@@
 			)
 		)
-		(property "Footprint" ""
+		(property "Footprint" "Capacitor_SMD:C_0603_1608Metric"
 			(at 204.1652 153.67 0)
 			(effects
@@
 			)
 		)
-		(property "Footprint" ""
+		(property "Footprint" "Connector_PinHeader_2.54mm:PinHeader_1x06_P2.54mm_Vertical"
 			(at 232.41 142.24 0)
 			(effects
@@
 			)
 		)
-		(property "Footprint" ""
+		(property "Footprint" "Connector_PinSocket_2.54mm:PinSocket_1x15_P2.54mm_Vertical"
 			(at 162.56 114.3 0)
 			(effects
@@
 			)
 		)
-		(property "Footprint" ""
+		(property "Footprint" "Connector_PinHeader_2.54mm:PinHeader_1x04_P2.54mm_Vertical"
 			(at 232.41 121.92 0)
 			(effects
@@
 			)
 		)
-		(property "Footprint" ""
+		(property "Footprint" "Resistor_SMD:R_0603_1608Metric"
 			(at 209.804 105.664 90)
 			(effects
@@
 			)
 		)
-		(property "Footprint" ""
+		(property "Footprint" "TestPoint:TestPoint_Pad_D1.5mm"
 			(at 132.08 130.81 0)
 			(effects
@@
 			)
 		)
-		(property "Footprint" ""
+		(property "Footprint" "TestPoint:TestPoint_Loop_D2.50mm_Drill1.0mm"
 			(at 132.08 104.14 0)
 			(effects
@@
 			)
 		)
-		(property "Footprint" ""
+		(property "Footprint" "Capacitor_SMD:C_0603_1608Metric"
 			(at 253.6952 139.7 0)
 			(effects
@@
 			)
 		)
-		(property "Footprint" ""
+		(property "Footprint" "TestPoint:TestPoint_Loop_D2.50mm_Drill1.0mm"
 			(at 132.08 113.03 0)
 			(effects
@@
 			)
 		)
-		(property "Footprint" ""
+		(property "Footprint" "TestPoint:TestPoint_Pad_D1.5mm"
 			(at 132.08 121.92 0)
 			(effects
