File: hardware/wearable_revB/wearable_revB.kicad_sch (KiCad schematic)
At the start: 15 parts, among them J1 Conn_01x15_Socket, J2 Conn_01x15_Socket, U1 MAX30102, U2 TMP117xxDRV

Commit message: Project Restart, debug and Platformio Setup
Parts:
- added J3: SSD1306 0.96" OLED, symbol Connector:Conn_01x04_Socket
- added U3: MPU-6050, Sensor_Motion:InvenSense_QFN-24_4x4mm_P0.5mm, symbol Sensor_Motion:MPU-6050
- J1: value Conn_01x15_Socket -> ESP32 LHS
- J2: value Conn_01x15_Socket -> ESP32 RHS
Connections:
- net 3.3V: now also J3.2 (Pin_2)
- net GND: now also J3.1 (Pin_1)
- net SCL: now also J2.14 (Pin_14), J3.3 (Pin_3)
- net SDA: now also J2.11 (Pin_11), J3.4 (Pin_4)
Other:
- moved on the sheet: J1, J2
