File: hardware/wearable_revB/wearable_revB/wearable_revB.kicad_sch (KiCad schematic)
At the start: 44 parts, among them J1 Conn_01x04, J2 USB_C_Receptacle, SW1 SW_Push, SW2 SW_Push, SW3 SW_Push, U1 TP4056-42-ESOP8, U2 ESP32-WROOM-32, U3 MAX30102, U4 AP2112K-1.8, U5 TMP117xxDRV, U6 MPU-6050

Commit message: Finalized PCB
Parts:
- added J3: Conn_01x02, custom:Battery_2Pin_THT, symbol Connector_Generic:Conn_01x02
- C1, C10, C11, C12, C13, C14, C15, C16, C17, C18, C2, C3, C4, C5, C6, C7, C8, C9: footprint (none) -> Capacitor_SMD:C_0603_1608Metric
- D1, D2: footprint (none) -> LED_SMD:LED_0603_1608Metric
- J1: footprint (none) -> Connector_PinHeader_1.27mm:PinHeader_1x04_P1.27mm_Vertical_SMD_Pin1Left
- J2: footprint (none) -> Connector_USB:USB_C_Receptacle_HRO_TYPE-C-31-M-12
- R1, R10, R11, R12, R2, R3, R4, R5, R6, R7, R8, R9: footprint (none) -> Resistor_SMD:R_0603_1608Metric
- SW1, SW2: footprint (none) -> Button_Switch_SMD:SW_SPST_B3U-1000P
- SW3: footprint (none) -> Button_Switch_SMD:SW_SPST_B3S-1100
- U7: footprint (none) -> custom:EASTRISING_ER-CON50HT-1
Connections:
- net BAT+: now also J3.1 (Pin_1)
- net GND: now also J3.2 (Pin_2)
- net MAX_INT: now also U2.6 (IO34)
- net VCC_5V: now reaches C1.1, J2.A4 (VBUS), J2.A9 (VBUS), J2.B4 (VBUS), J2.B9 (VBUS), R4.1, R5.1, R6.1, U1.4 (V_{CC})
- no-connect marks 0 -> 52
Other:
- moved on the sheet: C4, C5, U4
